Commit message: feat(viewer,urdf): URDF GLB 米制单位修复 + 纹理工作流闭环
viewer 对 URDF 的 GLB 改走 unitScale=1(不再 ×1000),GLB 保持毫米、
靠 URDF <mesh scale="0.001"> 接米制关节,修复带关节偏移的多 link 缩在原点的老 bug。
CAD/STEP 路径仍默认 unitScale=1000,不受影响。

配套:
- stl_to_wood_glb.py / texturize_urdf.py 默认改毫米(scale=1.0 + 改写引用写 scale=0.001)
- textures.md / 示例 README / 顶层 README 同步新单位约定
- viewer 前端重构建,engines/cad/dist 同步
- .gitignore 忽略 verify_urdf.py 的 _verify/ 临时截图

Generated with [Claude Code](https://claude.ai/code)
via [Happy](https://happy.engineering)

Co-Authored-By: Claude <noreply@anthropic.com>
Co-Authored-By: Happy <yesreply@happy.engineering>

File: skills/urdf/references/examples/wood-planetary/planetary_wood.urdf (robot description, URDF)
Before this commit: robot planetary_gear_wood, 6 links, 5 joints
Links:
- link carrier: geometry collision mesh filename=wood_meshes/carrier.glb scale=0.001 0.001 0.001; visual mesh filename=wood_meshes/carrier.glb scale=0.001 0.001 0.001
- link planet_1: geometry collision mesh filename=wood_meshes/planet_1.glb scale=0.001 0.001 0.001; visual mesh filename=wood_meshes/planet_1.glb scale=0.001 0.001 0.001
- link planet_2: geometry collision mesh filename=wood_meshes/planet_2.glb scale=0.001 0.001 0.001; visual mesh filename=wood_meshes/planet_2.glb scale=0.001 0.001 0.001
- link planet_3: geometry collision mesh filename=wood_meshes/planet_3.glb scale=0.001 0.001 0.001; visual mesh filename=wood_meshes/planet_3.glb scale=0.001 0.001 0.001
- link ring: geometry collision mesh filename=wood_meshes/ring.glb scale=0.001 0.001 0.001; visual mesh filename=wood_meshes/ring.glb scale=0.001 0.001 0.001
- link sun: geometry collision mesh filename=wood_meshes/sun.glb scale=0.001 0.001 0.001; visual mesh filename=wood_meshes/sun.glb scale=0.001 0.001 0.001
